File: KicadProject/LineFollower Project - RCX/LineFollowerRCX/LineFollowerRCX.kicad_pcb (KiCad board)
At the start: 2 copper layers, 100 x 70.9 mm, 13 parts, among them J1 Conn_01x11_Pin, J10 GND pinos, J2 Motor 1, J3 Motor 1, J4 Modulo bluetooth, J7 Conector sensor lateral Esque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, J8 Conector sensor lateral Direi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, J9 VCC pinos, U1 ROB-14450, U2 LM7805_TO220

Commit message: Arrumando design
Parts:
- moved J3 9.72 mm to (144.3, 146.5)
- moved J2 7.30 mm to (175.0, 145.3)
Routing:
- net Net-(J3--): track 39.6 -> 25.1 mm
- net Net-(J3-+): track 32.8 -> 19.4 mm
- net Net-(J2--): track 32.4 -> 21.5 mm
- net Net-(J2-+): track 22.6 -> 13.1 mm
- net Net-(U1-VM): track 68.4 -> 66.4 mm
- net Net-(Bateria1-+): track 31.6 -> 32.1 mm
- net (no net): vias 0 -> 8
- removed copper zone on F.Cu, net GND
